File: eagle/Platine.brd (EAGLE design)
At the start: 100 x 80 mm, 32 parts, among them IC3 7805, Q2 20MHz, X3 MA2X3

Commit message: 14 bridges
Parts:
- moved C2 6.48 mm to (50.8, 61.0)
- moved S2 5.85 mm to (55.9, 69.2), turned to 180 degrees
- moved LATCH 5.08 mm to (48.3, 47.0)
- moved R1 4.58 mm to (17.8, 68.6)
- moved R2 4.49 mm to (70.5, 73.0)
- moved C10 4.45 mm to (50.8, 31.1)
- moved C3 3.81 mm to (72.4, 68.6)
- moved ADRDEC 3.81 mm to (48.3, 16.5)
- moved R3 3.59 mm to (81.3, 69.8)
- moved X3 2.84 mm to (7.62, 41.9), turned to 90 degrees
- moved C9 2.54 mm to (76.2, 64.8), turned to 180 degrees
- moved C8 2.54 mm to (34.3, 63.5), turned to 180 degrees
- moved X4 1.80 mm to (15.2, 43.2)
- moved AD 1.27 mm to (7.62, 58.4)
- moved KEY 1.27 mm to (7.62, 22.9)
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Connections:
- net N$35: now also ADRDEC.16; no longer ADRDEC.18
Routing:
- net GND: track 125.9 -> 458.7 mm, vias 0 -> 6
- net +5V: track 19.9 -> 297.6 mm, vias 0 -> 10
- net N$3: track 0.00 -> 148.5 mm
- net 2PORT10: track 78.7 -> 0.00 mm
- net N$13: track 14.8 -> 47.8 mm
- net N$12: track 0.00 -> 31.3 mm, vias 0 -> 2
- net 2PORT9: track 42.5 -> 70.1 mm
- net 2PORT8: track 42.5 -> 68.9 mm
- net N$41: track 0.00 -> 23.4 mm
- net N$11: track 0.00 -> 20.4 mm
- net N$10: track 0.00 -> 17.8 mm
- net N$33: track 61.5 -> 47.9 mm
- net N$34: track 13.6 -> 0.00 mm
- net 1PORT1: track 80.8 -> 92.4 mm
- net N$32: track 37.1 -> 25.8 mm
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
Commit message: 4 remaining
Connections:
- net N$32: now also ADRDEC.2; no longer ADRDEC.5
- net N$33: now also ADRDEC.1; no longer ADRDEC.4
- net N$35: now also ADRDEC.12; no longer ADRDEC.16
- net N$36: now also ADRDEC.13; no longer ADRDEC.17
Routing:
- net N$34: track 0.00 -> 75.0 mm
- net 2PORT10: track 0.00 -> 47.5 mm
- net 2PORT11: track 0.00 -> 46.7 mm
- net N$33: track 47.9 -> 20.1 mm
- net N$41: track 23.4 -> 0.00 mm
- net +5V: track 297.6 -> 320.8 mm
- net N$32: track 25.8 -> 39.3 mm
- net N$35: track 58.1 -> 63.8 mm
- net N$36: track 53.5 -> 59.0 mm
- net N$12: track 31.3 -> 34.3 mm
- net 1PORT2: track 100.1 -> 98.0 mm
- net 1PORT1: track 92.4 -> 90.3 mm
- net GND: track 458.7 -> 459.3 mm
