File: eagle/Platine.brd (EAGLE design)
At the start: 100 x 80 mm, 32 parts, among them IC3 7805, Q2 20MHz, X3 MA2X3

Commit message: quick fix
Routing:
- net +5V: track 321.3 -> 322.9 mm
Changed lines of the file:
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@@
 <wire x1="7.9071125" y1="72.4408" x2="13.5713125" y2="78.105" width="1.27" layer="1"/>
 <wire x1="2.1082" y1="66.8782" x2="7.6708" y2="72.4408" width="1.27" layer="1"/>
-<wire x1="80.54763125" y1="78.105" x2="83.0072" y2="75.64543125" width="1.27" layer="1"/>
-<wire x1="83.0072" y1="64.9478" x2="83.185" y2="64.77" width="1.27" layer="1"/>
-<wire x1="83.0072" y1="75.64543125" x2="83.0072" y2="64.9478" width="1.27" layer="1"/>
-<wire x1="83.185" y1="64.77" x2="81.28" y2="64.77" width="1.27" layer="1"/>
-<wire x1="13.5713125" y1="78.105" x2="80.54763125" y2="78.105" width="1.27" layer="1"/>
+<wire x1="81.18263125" y1="78.105" x2="83.6422" y2="75.64543125" width="1.27" layer="1"/>
+<wire x1="83.6422" y1="75.64543125" x2="83.6422" y2="66.4972" width="1.27" layer="1"/>
+<wire x1="83.6422" y1="66.4972" x2="81.915" y2="64.77" width="1.27" layer="1"/>
+<wire x1="81.28" y1="64.77" x2="81.915" y2="64.77" width="1.27" layer="1"/>
+<wire x1="13.5713125" y1="78.105" x2="81.18263125" y2="78.105" width="1.27" layer="1"/>
 <wire x1="90.17" y1="58.42" x2="90.17" y2="55.88" width="1.27" layer="1"/>
 </signal>
@@
 <via x="13.335" y="73.66" extent="1-16" drill="0.6096"/>
 <wire x1="71.12" y1="68.58" x2="71.12" y2="66.675" width="1.27" layer="1"/>
-<wire x1="67.1322" y1="73.74043125" x2="66.12043125" y2="74.7522" width="1.27" layer="1"/>
-<wire x1="71.12" y1="68.58" x2="67.1322" y2="72.5678" width="1.27" layer="1"/>
-<wire x1="67.1322" y1="72.5678" x2="67.1322" y2="73.74043125" width="1.27" layer="1"/>
+<wire x1="71.12" y1="72.39" x2="68.7578" y2="74.7522" width="1.27" layer="1"/>
+<wire x1="71.12" y1="68.58" x2="71.12" y2="72.39" width="1.27" layer="1"/>
 <wire x1="17.9578" y1="74.7522" x2="17.78" y2="74.295" width="1.27" layer="1"/>
-<wire x1="66.12043125" y1="74.7522" x2="59.055" y2="74.7522" width="1.27" layer="1"/>
+<wire x1="68.7578" y1="74.7522" x2="59.055" y2="74.7522" width="1.27" layer="1"/>
 <wire x1="59.055" y1="74.7522" x2="55.245" y2="74.7522" width="1.27" layer="1"/>
 <wire x1="55.245" y1="74.7522" x2="38.1" y2="74.7522" width="1.27" layer="1"/>
@@
 <wire x1="22.3012" y1="65.23293125" x2="22.95586875" y2="65.8876" width="0.4064" layer="1"/>
 <wire x1="7.4676" y1="62.3824" x2="3.81" y2="62.3824" width="0.4064" layer="1"/>
-<wire x1="69.32039375" y1="73.025" x2="75.565" y2="73.025" width="0.4064" layer="1"/>
 <wire x1="15.24" y1="45.72" x2="17.9324" y2="48.4124" width="0.4064" layer="1"/>
 <wire x1="17.9324" y1="48.4124" x2="21.49413125" y2="48.4124" width="0.4064" layer="1"/>
 <wire x1="7.4676" y1="66.19813125" x2="7.4676" y2="62.3824" width="0.4064" layer="1"/>
-<wire x1="66.37399375" y1="75.9714" x2="69.32039375" y2="73.025" width="0.4064" layer="1"/>
-<wire x1="13.335" y1="75.9714" x2="66.37399375" y2="75.9714" width="0.4064" layer="1"/>
+<wire x1="75.565" y1="73.025" x2="75.565" y2="73.76539375" width="0.4064" layer="1"/>
+<wire x1="75.565" y1="73.76539375" x2="73.35899375" y2="75.9714" width="0.4064" layer="1"/>
+<wire x1="13.335" y1="75.9714" x2="73.35899375" y2="75.9714" width="0.4064" layer="1"/>
 <wire x1="3.81" y1="62.3824" x2="3.81" y2="66.8777625" width="0.4064" layer="1"/>
 <wire x1="25.9588" y1="67.77293125" x2="25.30413125" y2="68.4276" width="0.4064" layer="1"/>
