File: eagle/Platine.sch (EAGLE design)
At the start: 32 parts, among them IC3 7805, Q2 20MHz, X3 MA2X3

Commit message: na
Connections:
- net 2PORT8: now also ADRDEC.I8; no longer ADRDEC.I0/CLK
- net 2PORT9: now also ADRDEC.I7; no longer ADRDEC.I1
- net N$32: now also ADRDEC.I4; no longer ADRDEC.I2

Commit message: 14 bridges
Connections:
- net N$35: now also ADRDEC.IOQ3; no longer ADRDEC.IOQ1
Changed lines of the file:
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@@
 <net name="N$35" class="0">
 <segment>
-<pinref part="ADRDEC" gate="G$1" pin="IOQ1"/>
-<wire x1="195.58" y1="-58.42" x2="261.62" y2="-58.42" width="0.1524" layer="91"/>
 <wire x1="261.62" y1="-58.42" x2="261.62" y2="-5.08" width="0.1524" layer="91"/>
 <pinref part="LED" gate="G$1" pin="4"/>
 <wire x1="261.62" y1="-5.08" x2="266.7" y2="-5.08" width="0.1524" layer="91"/>
+<wire x1="261.62" y1="-58.42" x2="200.66" y2="-58.42" width="0.1524" layer="91"/>
+<wire x1="200.66" y1="-58.42" x2="200.66" y2="-63.5" width="0.1524" layer="91"/>
+<pinref part="ADRDEC" gate="G$1" pin="IOQ3"/>
+<wire x1="200.66" y1="-63.5" x2="195.58" y2="-63.5" width="0.1524" layer="91"/>
 </segment>
 </net>
 <net name="N$36" class="0">
 <segment>
-<pinref part="ADRDEC" gate="G$1" pin="IOQ2"/>
-<wire x1="195.58" y1="-60.96" x2="264.16" y2="-60.96" width="0.1524" layer="91"/>
 <wire x1="264.16" y1="-60.96" x2="264.16" y2="-7.62" width="0.1524" layer="91"/>
 <pinref part="LED" gate="G$1" pin="2"/>
 <wire x1="264.16" y1="-7.62" x2="266.7" y2="-7.62" width="0.1524" layer="91"/>
+<pinref part="ADRDEC" gate="G$1" pin="IOQ2"/>
+<wire x1="264.16" y1="-60.96" x2="195.58" y2="-60.96" width="0.1524" layer="91"/>
 </segment>
 </net>

Commit message: 4 remaining
Connections:
- net N$32: now also ADRDEC.I1; no longer ADRDEC.I4
- net N$33: now also ADRDEC.I0/CLK; no longer ADRDEC.I3
- net N$35: now also ADRDEC.IOQ7; no longer ADRDEC.IOQ3
- net N$36: now also ADRDEC.IOQ6; no longer ADRDEC.IOQ2
Changed lines of the file:
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@@
 <pinref part="RAM" gate="G$1" pin="\!OE"/>
 <wire x1="198.12" y1="-20.32" x2="208.28" y2="-20.32" width="0.1524" layer="91"/>
-<wire x1="147.32" y1="-40.64" x2="147.32" y2="-66.04" width="0.1524" layer="91"/>
+<pinref part="ADRDEC" gate="G$1" pin="I1"/>
+<wire x1="147.32" y1="-40.64" x2="147.32" y2="-58.42" width="0.1524" layer="91"/>
+<wire x1="147.32" y1="-58.42" x2="167.64" y2="-58.42" width="0.1524" layer="91"/>
 <junction x="147.32" y="-40.64"/>
-<pinref part="ADRDEC" gate="G$1" pin="I4"/>
-<wire x1="147.32" y1="-66.04" x2="167.64" y2="-66.04" width="0.1524" layer="91"/>
 </segment>
 </net>
@@
 <pinref part="RAM" gate="G$1" pin="\!WE"/>
 <wire x1="200.66" y1="-22.86" x2="208.28" y2="-22.86" width="0.1524" layer="91"/>
-<wire x1="144.78" y1="-43.18" x2="144.78" y2="-63.5" width="0.1524" layer="91"/>
+<pinref part="ADRDEC" gate="G$1" pin="I0/CLK"/>
+<wire x1="144.78" y1="-43.18" x2="144.78" y2="-55.88" width="0.1524" layer="91"/>
+<wire x1="144.78" y1="-55.88" x2="167.64" y2="-55.88" width="0.1524" layer="91"/>
 <junction x="144.78" y="-43.18"/>
-<pinref part="ADRDEC" gate="G$1" pin="I3"/>
-<wire x1="144.78" y1="-63.5" x2="167.64" y2="-63.5" width="0.1524" layer="91"/>
 </segment>
 </net>
@@
 <wire x1="261.62" y1="-5.08" x2="266.7" y2="-5.08" width="0.1524" layer="91"/>
 <wire x1="261.62" y1="-58.42" x2="200.66" y2="-58.42" width="0.1524" layer="91"/>
-<wire x1="200.66" y1="-58.42" x2="200.66" y2="-63.5" width="0.1524" layer="91"/>
-<pinref part="ADRDEC" gate="G$1" pin="IOQ3"/>
-<wire x1="200.66" y1="-63.5" x2="195.58" y2="-63.5" width="0.1524" layer="91"/>
+<pinref part="ADRDEC" gate="G$1" pin="IOQ7"/>
+<wire x1="195.58" y1="-73.66" x2="200.66" y2="-73.66" width="0.1524" layer="91"/>
+<wire x1="200.66" y1="-73.66" x2="200.66" y2="-58.42" width="0.1524" layer="91"/>
 </segment>
 </net>
 <net name="N$36" class="0">
 <segment>
-<wire x1="264.16" y1="-60.96" x2="264.16" y2="-7.62" width="0.1524" layer="91"/>
+<wire x1="264.16" y1="-71.12" x2="264.16" y2="-7.62" width="0.1524" layer="91"/>
 <pinref part="LED" gate="G$1" pin="2"/>
 <wire x1="264.16" y1="-7.62" x2="266.7" y2="-7.62" width="0.1524" layer="91"/>
-<pinref part="ADRDEC" gate="G$1" pin="IOQ2"/>
-<wire x1="264.16" y1="-60.96" x2="195.58" y2="-60.96" width="0.1524" layer="91"/>
+<pinref part="ADRDEC" gate="G$1" pin="IOQ6"/>
+<wire x1="264.16" y1="-71.12" x2="195.58" y2="-71.12" width="0.1524" layer="91"/>
 </segment>
 </net>
