File: eagle/Platine.sch (EAGLE design)
At the start: 32 parts, among them IC3 7805, Q2 20MHz, X3 MA2X3

Commit message: quick fix
Connections:
- net 2PORT8: now also ADRDEC.I8; no longer ADRDEC.I0/CLK
- net 2PORT9: now also ADRDEC.I7; no longer ADRDEC.I1
- net N$32: now also ADRDEC.I1; no longer ADRDEC.I2
- net N$33: now also ADRDEC.I0/CLK; no longer ADRDEC.I3
- net N$35: now also ADRDEC.IOQ7; no longer ADRDEC.IOQ1
- net N$36: now also ADRDEC.IOQ6; no longer ADRDEC.IOQ2
